Commit message: adding all experimental data and stats python files

File: src/data/jaco.urdf (robot description, URDF)
Before this commit: robot j2s7s300, 12 links, 11 joints
Links:
- added link j2s7s300_link_finger_tip_1; collision mesh filename=package://kinova_description/meshes/finger_distal.dae; visual mesh filename=package://kinova_description/meshes/finger_distal.dae
- added link j2s7s300_link_finger_tip_2; collision mesh filename=package://kinova_description/meshes/finger_distal.dae; visual mesh filename=package://kinova_description/meshes/finger_distal.dae
- added link j2s7s300_link_finger_tip_3; collision mesh filename=package://kinova_description/meshes/finger_distal.dae; visual mesh filename=package://kinova_description/meshes/finger_distal.dae
Joints:
- added joint j2s7s300_joint_finger_tip_1: type fixed, parent j2s7s300_link_finger_1, child j2s7s300_link_finger_tip_1, origin xyz=0.044 -0.003 0 rpy=0 0 0, axis 0 0 1, limit lower=0 upper=2 effort=30 velocity=5
- added joint j2s7s300_joint_finger_tip_2: type fixed, parent j2s7s300_link_finger_2, child j2s7s300_link_finger_tip_2, origin xyz=0.044 -0.003 0 rpy=0 0 0, axis 0 0 1, limit lower=0 upper=2 effort=30 velocity=5
- added joint j2s7s300_joint_finger_tip_3: type fixed, parent j2s7s300_link_finger_3, child j2s7s300_link_finger_tip_3, origin xyz=0.044 -0.003 0 rpy=0 0 0, axis 0 0 1, limit lower=0 upper=2 effort=30 velocity=5
